File: W5500.sch (KiCad schematic (older format))
At the start: 50 parts, among them P301 J1B1211CCD, SW301 SW_Push, U301 W5500, Y301 25Mhz

Commit message: connecting spi lines and cleaning-up I/O
Parts:
- L301: footprint (none) -> Resistors_SMD:R_1812; Characteristics (none) -> Ethernet; Critical (none) -> Y; Description (none) -> FERRITE BEAD 120 OHM 1812 1LN; MFN (none) -> Wurth Electronics; MPN (none) -> 742792511; Notes (none) -> X; Package ID (none) -> 1812; Source (none) -> Digikey
Changed lines of the file:
@@
 F 0 "L301" V 6600 1050 50  0000 C CNN
 F 1 "L" V 6725 1050 50  0000 C CNN
-F 2 "" H 6650 1050 50  0001 C CNN
-F 3 "" H 6650 1050 50  0001 C CNN
+F 2 "Resistors_SMD:R_1812" H 6650 1050 50  0001 C CNN
+F 3 "http://katalog.we-online.de/pbs/datasheet/742792511.pdf" H 6650 1050 50  0001 C CNN
+F 4 "742792511" H 6650 1050 60  0001 C CNN "MPN"
+F 5 "Wurth Electronics" H 6650 1050 60  0001 C CNN "MFN"
+F 6 "Ethernet" H 6650 1050 60  0001 C CNN "Characteristics"
+F 7 "FERRITE BEAD 120 OHM 1812 1LN" H 6650 1050 60  0001 C CNN "Description"
+F 8 "1812" H 6650 1050 60  0001 C CNN "Package ID"
+F 9 "Digikey" H 6650 1050 60  0001 C CNN "Source"
+F 10 "Y" H 6650 1050 60  0001 C CNN "Critical"
+F 11 "X" H 6650 1050 60  0001 C CNN "Notes"
 	1    6650 1050
 	1    0    0    -1

Commit message: more tweaks
Connections:
- net GND renamed GNDD
Changed lines of the file:
@@
 $Descr A4 11693 8268
 encoding utf-8
-Sheet 3 3
+Sheet 2 3
 Title ""
 Date ""
@@
 $EndComp
 $Comp
-L GND #PWR318
-U 1 1 5935BB41
-P 6800 4500
-F 0 "#PWR318" H 6800 4250 50  0001 C CNN
-F 1 "GND" H 6800 4350 50  0000 C CNN
-F 2 "" H 6800 4500 50  0001 C CNN
-F 3 "" H 6800 4500 50  0001 C CNN
-	1    6800 4500
-	1    0    0    -1
-$EndComp
-$Comp
 L C_Small C316
 U 1 1 5935C0D3
@@
 $EndComp
 $Comp
-L GND #PWR322
-U 1 1 5935C32E
-P 8750 1950
-F 0 "#PWR322" H 8750 1700 50  0001 C CNN
-F 1 "GND" H 8750 1800 50  0000 C CNN
-F 2 "" H 8750 1950 50  0001 C CNN
-F 3 "" H 8750 1950 50  0001 C CNN
-	1    8750 1950
-	1    0    0    -1
-$EndComp
-$Comp
-L GND #PWR319
-U 1 1 5935CA4B
-P 7050 4500
-F 0 "#PWR319" H 7050 4250 50  0001 C CNN
-F 1 "GND" H 7050 4350 50  0000 C CNN
-F 2 "" H 7050 4500 50  0001 C CNN
-F 3 "" H 7050 4500 50  0001 C CNN
-	1    7050 4500
-	1    0    0    -1
-$EndComp
-$Comp
 L R_Small R315
 U 1 1 5935CB13
@@
 $EndComp
 $Comp
-L GND #PWR316
-U 1 1 5935CFEA
-P 6400 2400
-F 0 "#PWR316" H 6400 2150 50  0001 C CNN
-F 1 "GND" H 6400 2250 50  0000 C CNN
-F 2 "" H 6400 2400 50  0001 C CNN
-F 3 "" H 6400 2400 50  0001 C CNN
-	1    6400 2400
-	1    0    0    -1
-$EndComp
-$Comp
 L L L301
 U 1 1 5935D6D3
@@
 F 11 "X" H 8750 3900 60  0001 C CNN "Notes"
 	1    8750 3900
-	1    0    0    -1
-$EndComp
-$Comp
-L GND #PWR323
-U 1 1 5935E848
-P 8750 4150
-F 0 "#PWR323" H 8750 3900 50  0001 C CNN
-F 1 "GND" H 8750 4000 50  0000 C CNN
-F 2 "" H 8750 4150 50  0001 C CNN
-F 3 "" H 8750 4150 50  0001 C CNN
-	1    8750 4150
 	1    0    0    -1
 $EndComp
@@
 $EndComp
 $Comp
-L GND #PWR320
-U 1 1 5935FDA9
-P 7900 4450
-F 0 "#PWR320" H 7900 4200 50  0001 C CNN
-F 1 "GND" H 7900 4300 50  0000 C CNN
-F 2 "" H 7900 4450 50  0001 C CNN
-F 3 "" H 7900 4450 50  0001 C CNN
-	1    7900 4450
-	1    0    0    -1
-$EndComp
-$Comp
-L GND #PWR325
-U 1 1 5936020E
-P 9050 5050
-F 0 "#PWR325" H 9050 4800 50  0001 C CNN
-F 1 "GND" H 9050 4900 50  0000 C CNN
-F 2 "" H 9050 5050 50  0001 C CNN
-F 3 "" H 9050 5050 50  0001 C CNN
-	1    9050 5050
-	1    0    0    -1
-$EndComp
-$Comp
 L C_Small C307
 U 1 1 5936211E
@@
 	1    0    0    -1
 $EndComp
-$Comp
-L GND #PWR312
-U 1 1 5936243F
-P 5250 5500
-F 0 "#PWR312" H 5250 5250 50  0001 C CNN
-F 1 "GND" H 5250 5350 50  0000 C CNN
-F 2 "" H 5250 5500 50  0001 C CNN
-F 3 "" H 5250 5500 50  0001 C CNN
-	1    5250 5500
-	1    0    0    -1
-$EndComp
-$Comp
-L GND #PWR314
-U 1 1 59362577
-P 5650 5500
-F 0 "#PWR314" H 5650 5250 50  0001 C CNN
-F 1 "GND" H 5650 5350 50  0000 C CNN
-F 2 "" H 5650 5500 50  0001 C CNN
-F 3 "" H 5650 5500 50  0001 C CNN
-	1    5650 5500
-	1    0    0    -1
-$EndComp
-$Comp
-L GND #PWR315
-U 1 1 593627C4
-P 5850 5500
-F 0 "#PWR315" H 5850 5250 50  0001 C CNN
-F 1 "GND" H 5850 5350 50  0000 C CNN
-F 2 "" H 5850 5500 50  0001 C CNN
-F 3 "" H 5850 5500 50  0001 C CNN
-	1    5850 5500
-	1    0    0    -1
-$EndComp
 NoConn ~ 5450 4600
 NoConn ~ 4850 4600
-$Comp
-L GND #PWR311
-U 1 1 5936312F
-P 5050 5500
-F 0 "#PWR311" H 5050 5250 50  0001 C CNN
-F 1 "GND" H 5050 5350 50  0000 C CNN
-F 2 "" H 5050 5500 50  0001 C CNN
-F 3 "" H 5050 5500 50  0001 C CNN
-	1    5050 5500
-	1    0    0    -1
-$EndComp
 $Comp
 L +3V3 #PWR326
@@
 Text Label 3600 5000 0    60   ~ 0
 ACTLED
-$Comp
-L GND #PWR306
-U 1 1 59365BEC
-P 3850 4200
-F 0 "#PWR306" H 3850 3950 50  0001 C CNN
-F 1 "GND" H 3850 4050 50  0000 C CNN
-F 2 "" H 3850 4200 50  0001 C CNN
-F 3 "" H 3850 4200 50  0001 C CNN
-	1    3850 4200
-	1    0    0    -1
-$EndComp
 $Comp
 L +3V3 #PWR303
@@
 $EndComp
 $Comp
-L GND #PWR301
-U 1 1 5936C6E4
-P 1950 6300
-F 0 "#PWR301" H 1950 6050 50  0001 C CNN
-F 1 "GND" H 1950 6150 50  0000 C CNN
-F 2 "" H 1950 6300 50  0001 C CNN
-F 3 "" H 1950 6300 50  0001 C CNN
-	1    1950 6300
-	1    0    0    -1
-$EndComp
-$Comp
 L R R301
 U 1 1 5936CB3E
@@
 	1    0    0    -1
 $EndComp
-$Comp
-L GND #PWR302
-U 1 1 593720A4
-P 3100 1800
-F 0 "#PWR302" H 3100 1550 50  0001 C CNN
-F 1 "GND" H 3100 1650 50  0000 C CNN
-F 2 "" H 3100 1800 50  0001 C CNN
-F 3 "" H 3100 1800 50  0001 C CNN
-	1    3100 1800
-	1    0    0    -1
-$EndComp
 Wire Wire Line
 	7300 2800 9500 2800
@@
 	4600 1600 4600 1650
 Connection ~ 4800 1600
-$Comp
-L GND #PWR309
-U 1 1 59393497
-P 4600 1650
-F 0 "#PWR309" H 4600 1400 50  0001 C CNN
-F 1 "GND" H 4600 1500 50  0000 C CNN
-F 2 "" H 4600 1650 50  0001 C CNN
-F 3 "" H 4600 1650 50  0001 C CNN
-	1    4600 1650
-	1    0    0    -1
-$EndComp
 Wire Wire Line
 	5000 1650 5000 1600
@@
 Wire Wire Line
 	4700 5350 4700 5500
-$Comp
-L GND #PWR310
-U 1 1 59397767
-P 4700 5500
-F 0 "#PWR310" H 4700 5250 50  0001 C CNN
-F 1 "GND" H 4700 5350 50  0000 C CNN
-F 2 "" H 4700 5500 50  0001 C CNN
-F 3 "" H 4700 5500 50  0001 C CNN
-	1    4700 5500
-	1    0    0    -1
-$EndComp
 $Comp
 L R R326
@@
 	3800 1900 3800 2000
 $Comp
-L GND #PWR305
-U 1 1 5938A6BC
+L GNDD #PWR?
+U 1 1 593A0279
+P 8750 1950
+F 0 "#PWR?" H 8750 1700 50  0001 C CNN
+F 1 "GNDD" H 8750 1800 50  0000 C CNN
+F 2 "" H 8750 1950 50  0001 C CNN
+F 3 "" H 8750 1950 50  0001 C CNN
+	1    8750 1950
+	1    0    0    -1
+$EndComp
+$Comp
+L GNDD #PWR?
+U 1 1 593A0321
+P 9050 5050
+F 0 "#PWR?" H 9050 4800 50  0001 C CNN
+F 1 "GNDD" H 9050 4900 50  0000 C CNN
+F 2 "" H 9050 5050 50  0001 C CNN
+F 3 "" H 9050 5050 50  0001 C CNN
+	1    9050 5050
+	1    0    0    -1
+$EndComp
+$Comp
+L GNDD #PWR?
+U 1 1 593A045B
+P 7900 4450
+F 0 "#PWR?" H 7900 4200 50  0001 C CNN
+F 1 "GNDD" H 7900 4300 50  0000 C CNN
+F 2 "" H 7900 4450 50  0001 C CNN
+F 3 "" H 7900 4450 50  0001 C CNN
+	1    7900 4450
+	1    0    0    -1
+$EndComp
+$Comp
+L GNDD #PWR?
+U 1 1 593A04FC
+P 7050 4500
+F 0 "#PWR?" H 7050 4250 50  0001 C CNN
+F 1 "GNDD" H 7050 4350 50  0000 C CNN
+F 2 "" H 7050 4500 50  0001 C CNN
+F 3 "" H 7050 4500 50  0001 C CNN
+	1    7050 4500
+	1    0    0    -1
+$EndComp
+$Comp
+L GNDD #PWR?
+U 1 1 593A059D
+P 6800 4500
+F 0 "#PWR?" H 6800 4250 50  0001 C CNN
+F 1 "GNDD" H 6800 4350 50  0000 C CNN
+F 2 "" H 6800 4500 50  0001 C CNN
+F 3 "" H 6800 4500 50  0001 C CNN
+	1    6800 4500
+	1    0    0    -1
+$EndComp
+$Comp
+L GNDD #PWR?
+U 1 1 593A09C8
+P 5850 5500
+F 0 "#PWR?" H 5850 5250 50  0001 C CNN
+F 1 "GNDD" H 5850 5350 50  0000 C CNN
+F 2 "" H 5850 5500 50  0001 C CNN
+F 3 "" H 5850 5500 50  0001 C CNN
+	1    5850 5500
+	1    0    0    -1
+$EndComp
+$Comp
+L GNDD #PWR?
+U 1 1 593A0A69
+P 5650 5500
+F 0 "#PWR?" H 5650 5250 50  0001 C CNN
+F 1 "GNDD" H 5650 5350 50  0000 C CNN
+F 2 "" H 5650 5500 50  0001 C CNN
+F 3 "" H 5650 5500 50  0001 C CNN
+	1    5650 5500
+	1    0    0    -1
+$EndComp
+$Comp
+L GNDD #PWR?
+U 1 1 593A0B0A
+P 5250 5500
+F 0 "#PWR?" H 5250 5250 50  0001 C CNN
+F 1 "GNDD" H 5250 5350 50  0000 C CNN
+F 2 "" H 5250 5500 50  0001 C CNN
+F 3 "" H 5250 5500 50  0001 C CNN
+	1    5250 5500
+	1    0    0    -1
+$EndComp
+$Comp
+L GNDD #PWR?
+U 1 1 593A0BAB
+P 5050 5500
+F 0 "#PWR?" H 5050 5250 50  0001 C CNN
+F 1 "GNDD" H 5050 5350 50  0000 C CNN
+F 2 "" H 5050 5500 50  0001 C CNN
+F 3 "" H 5050 5500 50  0001 C CNN
+	1    5050 5500
+	1    0    0    -1
+$EndComp
+$Comp
+L GNDD #PWR?
+U 1 1 593A0C4C
+P 4700 5500
+F 0 "#PWR?" H 4700 5250 50  0001 C CNN
+F 1 "GNDD" H 4700 5350 50  0000 C CNN
+F 2 "" H 4700 5500 50  0001 C CNN
+F 3 "" H 4700 5500 50  0001 C CNN
+	1    4700 5500
+	1    0    0    -1
+$EndComp
+$Comp
+L GNDD #PWR?
+U 1 1 593A0F16
+P 6400 2400
+F 0 "#PWR?" H 6400 2150 50  0001 C CNN
+F 1 "GNDD" H 6400 2250 50  0000 C CNN
+F 2 "" H 6400 2400 50  0001 C CNN
+F 3 "" H 6400 2400 50  0001 C CNN
+	1    6400 2400
+	1    0    0    -1
+$EndComp
+$Comp
+L GNDD #PWR?
+U 1 1 593A0FB7
 P 3800 2000
-F 0 "#PWR305" H 3800 1750 50  0001 C CNN
-F 1 "GND" H 3800 1850 50  0000 C CNN
+F 0 "#PWR?" H 3800 1750 50  0001 C CNN
+F 1 "GNDD" H 3800 1850 50  0000 C CNN
 F 2 "" H 3800 2000 50  0001 C CNN
 F 3 "" H 3800 2000 50  0001 C CNN
@@
 	1    0    0    -1
 $EndComp
+$Comp
+L GNDD #PWR?
+U 1 1 593A1058
+P 3100 1800
+F 0 "#PWR?" H 3100 1550 50  0001 C CNN
+F 1 "GNDD" H 3100 1650 50  0000 C CNN
+F 2 "" H 3100 1800 50  0001 C CNN
+F 3 "" H 3100 1800 50  0001 C CNN
+	1    3100 1800
+	1    0    0    -1
+$EndComp
+$Comp
+L GNDD #PWR?
+U 1 1 593A112C
+P 4600 1650
+F 0 "#PWR?" H 4600 1400 50  0001 C CNN
+F 1 "GNDD" H 4600 1500 50  0000 C CNN
+F 2 "" H 4600 1650 50  0001 C CNN
+F 3 "" H 4600 1650 50  0001 C CNN
+	1    4600 1650
+	1    0    0    -1
+$EndComp
+$Comp
+L GNDD #PWR?
+U 1 1 593A12FA
+P 1950 6300
+F 0 "#PWR?" H 1950 6050 50  0001 C CNN
+F 1 "GNDD" H 1950 6150 50  0000 C CNN
+F 2 "" H 1950 6300 50  0001 C CNN
+F 3 "" H 1950 6300 50  0001 C CNN
+	1    1950 6300
+	1    0    0    -1
+$EndComp
+$Comp
+L GNDD #PWR?
+U 1 1 593A139B
+P 3850 4200
+F 0 "#PWR?" H 3850 3950 50  0001 C CNN
+F 1 "GNDD" H 3850 4050 50  0000 C CNN
+F 2 "" H 3850 4200 50  0001 C CNN
+F 3 "" H 3850 4200 50  0001 C CNN
+	1    3850 4200
+	1    0    0    -1
+$EndComp
+$Comp
+L GNDD #PWR?
+U 1 1 593A1889
+P 8750 4150
+F 0 "#PWR?" H 8750 3900 50  0001 C CNN
+F 1 "GNDD" H 8750 4000 50  0000 C CNN
+F 2 "" H 8750 4150 50  0001 C CNN
+F 3 "" H 8750 4150 50  0001 C CNN
+	1    8750 4150
+	1    0    0    -1
+$EndComp

Commit message: final design sent to fab
Connections:
- net X0: now also C301.1, Y301.3; no longer R301.1
- net XI/CLKN: now also R301.1; no longer C302.1, Y301.3
- net at R301.2, Y301.1: now also C302.1; no longer C301.1
Other:
- moved on the sheet: R301
Changed lines of the file:
@@
 U 1 1 5936BD03
 P 1950 5700
-F 0 "Y301" H 1750 6100 50  0000 L CNN
-F 1 "25Mhz" H 1750 6000 50  0000 L CNN
+F 0 "Y301" H 2050 5350 50  0000 L CNN
+F 1 "25Mhz" H 2000 5450 50  0000 L CNN
 F 2 "3ML_SMD_Generic:3ML_4-SMD" H 1950 5700 50  0001 C CNN
 F 3 "http://www.abracon.com/Resonators/ABM8G.pdf" H 1950 5700 50  0001 C CNN
@@
 F 11 "X" H 1950 5700 60  0001 C CNN "Notes"
 	1    1950 5700
-	1    0    0    -1
+	-1   0    0    1
 $EndComp
 $Comp
@@
 L R R301
 U 1 1 5936CB3E
-P 1550 5450
-F 0 "R301" V 1630 5450 50  0000 C CNN
-F 1 "0" V 1550 5450 50  0000 C CNN
-F 2 "Resistors_SMD:R_0805" V 1480 5450 50  0001 C CNN
-F 3 "http://www.yageo.com/documents/recent/PYu-RC_Group_51_RoHS_L_7.pdf" H 1550 5450 50  0001 C CNN
-F 4 "RC0805JR-070RL" H 1550 5450 60  0001 C CNN "MPN"
-F 5 "Yageo" H 1550 5450 60  0001 C CNN "MFN"
-F 6 "Ethernet" H 1550 5450 60  0001 C CNN "Characteristics"
-F 7 "RES SMD 0.0 OHM JUMPER 1/8W 0805" H 1550 5450 60  0001 C CNN "Description"
-F 8 "0805" H 1550 5450 60  0001 C CNN "Package ID"
-F 9 "Digikey" H 1550 5450 60  0001 C CNN "Source"
-F 10 "Y" H 1550 5450 60  0001 C CNN "Critical"
-F 11 "X" H 1550 5450 60  0001 C CNN "Notes"
-	1    1550 5450
+P 2350 5450
+F 0 "R301" V 2430 5450 50  0000 C CNN
+F 1 "0" V 2350 5450 50  0000 C CNN
+F 2 "Resistors_SMD:R_0805" V 2280 5450 50  0001 C CNN
+F 3 "http://www.yageo.com/documents/recent/PYu-RC_Group_51_RoHS_L_7.pdf" H 2350 5450 50  0001 C CNN
+F 4 "RC0805JR-070RL" H 2350 5450 60  0001 C CNN "MPN"
+F 5 "Yageo" H 2350 5450 60  0001 C CNN "MFN"
+F 6 "Ethernet" H 2350 5450 60  0001 C CNN "Characteristics"
+F 7 "RES SMD 0.0 OHM JUMPER 1/8W 0805" H 2350 5450 60  0001 C CNN "Description"
+F 8 "0805" H 2350 5450 60  0001 C CNN "Package ID"
+F 9 "Digikey" H 2350 5450 60  0001 C CNN "Source"
+F 10 "Y" H 2350 5450 60  0001 C CNN "Critical"
+F 11 "X" H 2350 5450 60  0001 C CNN "Notes"
+	1    2350 5450
 	1    0    0    -1
 $EndComp
@@
 	10050 4850 10550 4850
 Wire Wire Line
-	1800 5700 1550 5700
-Wire Wire Line
-	2350 5700 2100 5700
-Wire Wire Line
-	2350 5150 2350 5750
-Wire Wire Line
-	1550 5600 1550 5750
+	1550 4900 1550 5750
 Wire Wire Line
 	1550 5950 1550 6100
 Wire Wire Line
 	1550 6100 2350 6100
-Wire Wire Line
-	1950 5900 1950 6300
 Wire Wire Line
 	2350 6100 2350 5950
 Connection ~ 1950 6100
-Wire Wire Line
-	1950 5500 1950 5450
-Wire Wire Line
-	1950 5450 2200 5450
-Wire Wire Line
-	2200 5450 2200 6100
 Connection ~ 2200 6100
 Connection ~ 1550 5700
-Wire Wire Line
-	1550 4900 1550 5300
 Connection ~ 2350 5700
 Wire Wire Line
@@
 	1    0    0    -1
 $EndComp
+Wire Wire Line
+	1950 5900 1950 6300
+Wire Wire Line
+	1950 5500 1950 5400
+Wire Wire Line
+	1950 5400 2200 5400
+Wire Wire Line
+	2200 5400 2200 6100
+Wire Wire Line
+	2350 5600 2350 5750
+Wire Wire Line
+	2350 5300 2350 5150
+Wire Wire Line
+	1800 5700 1550 5700
+Wire Wire Line
+	2100 5700 2350 5700
 $EndSCHEMATC
