File: W5500.sch (KiCad schematic (older format))
At the start: 50 parts, among them P301 J1B1211CCD, SW301 SW_Push, U301 W5500, Y301 25Mhz

Commit message: updated for rev2 to go to OSHPark. Fixed footprints and changed topside routing to have better noise characteristics
Parts:
- Y301: footprint 3ML_SMD_Generic:3ML_4-SMD -> Oscillators:Oscillator_SMD_Abracon_ASE-4pin_3.2x2.5mm; Populate (none) -> 1
Changed lines of the file:
@@
 U 1 1 59359FF3
 P 10000 3500
+AR Path="/59359FF3" Ref="P301"  Part="1"
+AR Path="/5935977E/59359FF3" Ref="P301"  Part="1"
 F 0 "P301" H 9750 4400 60  0000 C CNN
 F 1 "J1B1211CCD" H 10000 2700 60  0000 C CNN
@@
 $EndComp
 $Comp
-L +3V3 #PWR217
+L +3V3 #PWR014
 U 1 1 5935BACE
 P 6650 850
-F 0 "#PWR217" H 6650 700 50  0001 C CNN
+F 0 "#PWR014" H 6650 700 50  0001 C CNN
 F 1 "+3V3" H 6650 990 50  0000 C CNN
 F 2 "" H 6650 850 50  0001 C CNN
@@
 $EndComp
 $Comp
-L +3V3 #PWR221
+L +3V3 #PWR015
 U 1 1 5935E15E
 P 8150 2200
-F 0 "#PWR221" H 8150 2050 50  0001 C CNN
+F 0 "#PWR015" H 8150 2050 50  0001 C CNN
 F 1 "+3V3" H 8150 2340 50  0000 C CNN
 F 2 "" H 8150 2200 50  0001 C CNN
@@
 NoConn ~ 4850 4600
 $Comp
-L +3V3 #PWR226
+L +3V3 #PWR016
 U 1 1 59363D0D
 P 9250 2200
-F 0 "#PWR226" H 9250 2050 50  0001 C CNN
+F 0 "#PWR016" H 9250 2050 50  0001 C CNN
 F 1 "+3V3" H 9250 2340 50  0000 C CNN
 F 2 "" H 9250 2200 50  0001 C CNN
@@
 ACTLED
 $Comp
-L +3V3 #PWR203
+L +3V3 #PWR017
 U 1 1 5936640D
 P 3150 2500
-F 0 "#PWR203" H 3150 2350 50  0001 C CNN
+F 0 "#PWR017" H 3150 2350 50  0001 C CNN
 F 1 "+3V3" H 3150 2640 50  0000 C CNN
 F 2 "" H 3150 2500 50  0001 C CNN
@@
 F 0 "Y301" H 1750 6100 50  0000 L CNN
 F 1 "25Mhz" H 1750 6000 50  0000 L CNN
-F 2 "3ML_SMD_Generic:3ML_4-SMD" H 1950 5700 50  0001 C CNN
+F 2 "Oscillators:Oscillator_SMD_Abracon_ASE-4pin_3.2x2.5mm" H 1950 5700 50  0001 C CNN
 F 3 "http://www.abracon.com/Resonators/ABM8G.pdf" H 1950 5700 50  0001 C CNN
-F 4 "ABM8G-25.000MHZ-18-D2Y-T" H 1950 5700 60  0001 C CNN "MPN"
-F 5 "Abracon LLC" H 1950 5700 60  0001 C CNN "MFN"
-F 6 "Ethernet" H 1950 5700 60  0001 C CNN "Characteristics"
-F 7 "CRYSTAL 25.0000MHZ 18PF SMD" H 1950 5700 60  0001 C CNN "Description"
-F 8 "4-SMD" H 1950 5700 60  0001 C CNN "Package ID"
-F 9 "Digikey" H 1950 5700 60  0001 C CNN "Source"
-F 10 "Y" H 1950 5700 60  0001 C CNN "Critical"
-F 11 "X" H 1950 5700 60  0001 C CNN "Notes"
+F 4 "Ethernet" H 1950 5700 60  0001 C CNN "Characteristics"
+F 5 "CRYSTAL 25.0000MHZ 18PF SMD" H 1950 5700 60  0001 C CNN "Description"
+F 6 "Abracon LLC" H 1950 5700 60  0001 C CNN "MFN"
+F 7 "4-SMD" H 1950 5700 60  0001 C CNN "Package ID"
+F 8 "Digikey" H 1950 5700 60  0001 C CNN "Source"
+F 9 "Y" H 1950 5700 60  0001 C CNN "Critical"
+F 10 "X" H 1950 5700 60  0001 C CNN "Notes"
+F 11 "1" H 1950 5700 60  0001 C CNN "Populate"
+F 12 "ABM8G-25.000MHZ-18-D2Y-T" H 1950 5700 60  0001 C CNN "MPN"
 	1    1950 5700
 	1    0    0    -1
@@
 Connection ~ 9050 4550
 $Comp
-L Earth #PWR224
+L Earth #PWR018
 U 1 1 5938C9B2
 P 8850 5050
-F 0 "#PWR224" H 8850 4800 50  0001 C CNN
+F 0 "#PWR018" H 8850 4800 50  0001 C CNN
 F 1 "Earth" H 8850 4900 50  0001 C CNN
 F 2 "" H 8850 5050 50  0001 C CNN
@@
 	4100 2550 4100 2450
 $Comp
-L +3V3 #PWR208
+L +3V3 #PWR019
 U 1 1 59390E7D
 P 4100 2450
-F 0 "#PWR208" H 4100 2300 50  0001 C CNN
+F 0 "#PWR019" H 4100 2300 50  0001 C CNN
 F 1 "+3V3" H 4100 2590 50  0000 C CNN
 F 2 "" H 4100 2450 50  0001 C CNN
@@
 Connection ~ 5500 1200
 $Comp
-L +3V3 #PWR213
+L +3V3 #PWR020
 U 1 1 5939589A
 P 5500 1100
-F 0 "#PWR213" H 5500 950 50  0001 C CNN
+F 0 "#PWR020" H 5500 950 50  0001 C CNN
 F 1 "+3V3" H 5500 1240 50  0000 C CNN
 F 2 "" H 5500 1100 50  0001 C CNN
@@
 	3900 2550 3900 2450
 $Comp
-L +3V3 #PWR207
+L +3V3 #PWR021
 U 1 1 59396583
 P 3900 2450
-F 0 "#PWR207" H 3900 2300 50  0001 C CNN
+F 0 "#PWR021" H 3900 2300 50  0001 C CNN
 F 1 "+3V3" H 3900 2590 50  0000 C CNN
 F 2 "" H 3900 2450 50  0001 C CNN
@@
 	3800 1200 3800 1100
 $Comp
-L +3V3 #PWR204
+L +3V3 #PWR022
 U 1 1 5938A31B
 P 3800 1100
-F 0 "#PWR204" H 3800 950 50  0001 C CNN
+F 0 "#PWR022" H 3800 950 50  0001 C CNN
 F 1 "+3V3" H 3800 1240 50  0000 C CNN
 F 2 "" H 3800 1100 50  0001 C CNN
@@
 	3800 1900 3800 2000
 $Comp
-L GNDD #PWR222
+L GNDD #PWR023
 U 1 1 593A0279
 P 8750 1950
-F 0 "#PWR222" H 8750 1700 50  0001 C CNN
+F 0 "#PWR023" H 8750 1700 50  0001 C CNN
 F 1 "GNDD" H 8750 1800 50  0000 C CNN
 F 2 "" H 8750 1950 50  0001 C CNN
@@
 $EndComp
 $Comp
-L GNDD #PWR225
+L GNDD #PWR024
 U 1 1 593A0321
 P 9050 5050
-F 0 "#PWR225" H 9050 4800 50  0001 C CNN
+F 0 "#PWR024" H 9050 4800 50  0001 C CNN
 F 1 "GNDD" H 9050 4900 50  0000 C CNN
 F 2 "" H 9050 5050 50  0001 C CNN
@@
 $EndComp
 $Comp
-L GNDD #PWR220
+L GNDD #PWR025
 U 1 1 593A045B
 P 7900 4450
-F 0 "#PWR220" H 7900 4200 50  0001 C CNN
+F 0 "#PWR025" H 7900 4200 50  0001 C CNN
 F 1 "GNDD" H 7900 4300 50  0000 C CNN
 F 2 "" H 7900 4450 50  0001 C CNN
@@
 $EndComp
 $Comp
-L GNDD #PWR219
+L GNDD #PWR026
 U 1 1 593A04FC
 P 7050 4500
-F 0 "#PWR219" H 7050 4250 50  0001 C CNN
+F 0 "#PWR026" H 7050 4250 50  0001 C CNN
 F 1 "GNDD" H 7050 4350 50  0000 C CNN
 F 2 "" H 7050 4500 50  0001 C CNN
@@
 $EndComp
 $Comp
-L GNDD #PWR218
+L GNDD #PWR027
 U 1 1 593A059D
 P 6800 4500
-F 0 "#PWR218" H 6800 4250 50  0001 C CNN
+F 0 "#PWR027" H 6800 4250 50  0001 C CNN
 F 1 "GNDD" H 6800 4350 50  0000 C CNN
 F 2 "" H 6800 4500 50  0001 C CNN
@@
 $EndComp
 $Comp
-L GNDD #PWR215
+L GNDD #PWR028
 U 1 1 593A09C8
 P 5850 5500
-F 0 "#PWR215" H 5850 5250 50  0001 C CNN
+F 0 "#PWR028" H 5850 5250 50  0001 C CNN
 F 1 "GNDD" H 5850 5350 50  0000 C CNN
 F 2 "" H 5850 5500 50  0001 C CNN
@@
 $EndComp
 $Comp
-L GNDD #PWR214
+L GNDD #PWR029
 U 1 1 593A0A69
 P 5650 5500
-F 0 "#PWR214" H 5650 5250 50  0001 C CNN
+F 0 "#PWR029" H 5650 5250 50  0001 C CNN
 F 1 "GNDD" H 5650 5350 50  0000 C CNN
 F 2 "" H 5650 5500 50  0001 C CNN
@@
 $EndComp
 $Comp
-L GNDD #PWR212
+L GNDD #PWR030
 U 1 1 593A0B0A
 P 5250 5500
-F 0 "#PWR212" H 5250 5250 50  0001 C CNN
+F 0 "#PWR030" H 5250 5250 50  0001 C CNN
 F 1 "GNDD" H 5250 5350 50  0000 C CNN
 F 2 "" H 5250 5500 50  0001 C CNN
@@
 $EndComp
 $Comp
-L GNDD #PWR211
+L GNDD #PWR031
 U 1 1 593A0BAB
 P 5050 5500
-F 0 "#PWR211" H 5050 5250 50  0001 C CNN
+F 0 "#PWR031" H 5050 5250 50  0001 C CNN
 F 1 "GNDD" H 5050 5350 50  0000 C CNN
 F 2 "" H 5050 5500 50  0001 C CNN
@@
 $EndComp
 $Comp
-L GNDD #PWR210
+L GNDD #PWR032
 U 1 1 593A0C4C
 P 4700 5500
-F 0 "#PWR210" H 4700 5250 50  0001 C CNN
+F 0 "#PWR032" H 4700 5250 50  0001 C CNN
 F 1 "GNDD" H 4700 5350 50  0000 C CNN
 F 2 "" H 4700 5500 50  0001 C CNN
@@
 $EndComp
 $Comp
-L GNDD #PWR216
+L GNDD #PWR033
 U 1 1 593A0F16
 P 6400 2400
-F 0 "#PWR216" H 6400 2150 50  0001 C CNN
+F 0 "#PWR033" H 6400 2150 50  0001 C CNN
 F 1 "GNDD" H 6400 2250 50  0000 C CNN
 F 2 "" H 6400 2400 50  0001 C CNN
@@
 $EndComp
 $Comp
-L GNDD #PWR205
+L GNDD #PWR034
 U 1 1 593A0FB7
 P 3800 2000
-F 0 "#PWR205" H 3800 1750 50  0001 C CNN
+F 0 "#PWR034" H 3800 1750 50  0001 C CNN
 F 1 "GNDD" H 3800 1850 50  0000 C CNN
 F 2 "" H 3800 2000 50  0001 C CNN
@@
 $EndComp
 $Comp
-L GNDD #PWR202
+L GNDD #PWR035
 U 1 1 593A1058
 P 3100 1800
-F 0 "#PWR202" H 3100 1550 50  0001 C CNN
+F 0 "#PWR035" H 3100 1550 50  0001 C CNN
 F 1 "GNDD" H 3100 1650 50  0000 C CNN
 F 2 "" H 3100 1800 50  0001 C CNN
@@
 $EndComp
 $Comp
-L GNDD #PWR209
+L GNDD #PWR036
 U 1 1 593A112C
 P 4600 1650
-F 0 "#PWR209" H 4600 1400 50  0001 C CNN
+F 0 "#PWR036" H 4600 1400 50  0001 C CNN
 F 1 "GNDD" H 4600 1500 50  0000 C CNN
 F 2 "" H 4600 1650 50  0001 C CNN
@@
 $EndComp
 $Comp
-L GNDD #PWR201
+L GNDD #PWR037
 U 1 1 593A12FA
 P 1950 6300
-F 0 "#PWR201" H 1950 6050 50  0001 C CNN
+F 0 "#PWR037" H 1950 6050 50  0001 C CNN
 F 1 "GNDD" H 1950 6150 50  0000 C CNN
 F 2 "" H 1950 6300 50  0001 C CNN
@@
 $EndComp
 $Comp
-L GNDD #PWR206
+L GNDD #PWR038
 U 1 1 593A139B
 P 3850 4200
-F 0 "#PWR206" H 3850 3950 50  0001 C CNN
+F 0 "#PWR038" H 3850 3950 50  0001 C CNN
 F 1 "GNDD" H 3850 4050 50  0000 C CNN
 F 2 "" H 3850 4200 50  0001 C CNN
@@
 $EndComp
 $Comp
-L GNDD #PWR223
+L GNDD #PWR039
 U 1 1 593A1889
 P 8750 4150
-F 0 "#PWR223" H 8750 3900 50  0001 C CNN
+F 0 "#PWR039" H 8750 3900 50  0001 C CNN
 F 1 "GNDD" H 8750 4000 50  0000 C CNN
 F 2 "" H 8750 4150 50  0001 C CNN

Commit message: fixing some component/BOM part numbers
Parts:
- SW301: MFN PTS645SK43SMTR92 LFS -> C&K; MPN C&K -> PTS645SK43SMTR92 LFS; Populate (none) -> 1
Changed lines of the file:
@@
 F 2 "Buttons_Switches_SMD:SW_SPST_PTS645" H 3400 1800 50  0001 C CNN
 F 3 "http://www.ckswitches.com/media/1471/pts645.pdf" H 3400 1800 50  0001 C CNN
-F 4 "C&K" H 3400 1600 60  0001 C CNN "MPN"
-F 5 "PTS645SK43SMTR92 LFS" H 3400 1600 60  0001 C CNN "MFN"
-F 6 "Ethernet" H 3400 1600 60  0001 C CNN "Characteristics"
-F 7 "SWITCH TACTILE SPST-NO 0.05A 12V" H 3400 1600 60  0001 C CNN "Description"
-F 8 "SMD" H 3400 1600 60  0001 C CNN "Package ID"
-F 9 "Digikey" H 3400 1600 60  0001 C CNN "Source"
-F 10 "Y" H 3400 1600 60  0001 C CNN "Critical"
-F 11 "X" H 3400 1600 60  0001 C CNN "Notes"
+F 4 "Ethernet" H 3400 1600 60  0001 C CNN "Characteristics"
+F 5 "SWITCH TACTILE SPST-NO 0.05A 12V" H 3400 1600 60  0001 C CNN "Description"
+F 6 "C&K" H 3400 1600 60  0001 C CNN "MFN"
+F 7 "SMD" H 3400 1600 60  0001 C CNN "Package ID"
+F 8 "Digikey" H 3400 1600 60  0001 C CNN "Source"
+F 9 "Y" H 3400 1600 60  0001 C CNN "Critical"
+F 10 "X" H 3400 1600 60  0001 C CNN "Notes"
+F 11 "1" H 3400 1600 60  0001 C CNN "Populate"
+F 12 "PTS645SK43SMTR92 LFS" H 3400 1600 60  0001 C CNN "MPN"
 	1    3400 1600
 	1    0    0    -1
